File: huey.kicad_pcb (KiCad board)
At the start: 2 copper layers, 0 parts

Commit message: starting layout
Parts:
- added P1: LED_HEADERS, Pin_Headers:Pin_Header_Straight_1x03, F.Cu at (83.2, 78.1)
- added Q1: MF-DSC-SOT233-BSS138, Huey:MF_Discrete_Semiconductor-SOT-23-3, F.Cu at (98.4, 95.9)
- added R1: MF-RES-0603-1K, Resistors_SMD:R_0603, F.Cu at (97.8, 91.4)
- added R2: MF-RES-0603-1K, Resistors_SMD:R_0603, F.Cu at (97.2, 99.7)
- added R3: MF-RES-0603-1K, Resistors_SMD:R_0603, F.Cu at (100.3, 91.4)
- added R4: MF-RES-0603-1K, Resistors_SMD:R_0603, F.Cu at (99.7, 99.7)
- added SD1: MF-MICROSD, Huey:MF_Connectors-MF-MICROSD, F.Cu at (62.9, 87.0)
- added U1: ADAFRUIT_FEATHER_M0_WIFI, Huey:Adafruit_Feather_M0_WiFi, F.Cu at (83.2, 80.0)
Other:
- board outline added: 50 x 50 mm
