File: huey.kicad_pcb (KiCad board)
At the start: 2 copper layers, 50 x 50 mm, 8 parts, among them P1 LED_HEADERS, Q1 MF-DSC-SOT233-BSS138, U1 ADAFRUIT_FEATHER_M0_WIFI

Commit message: WIP
Parts:
- added C1: MF-CAP-6.3MM-100uF, Huey:MF_Passives-CP6.3MM, F.Cu at (117.5, 74.3)
- added CON1: BARREL_JACK, Huey:PJ-036AH-SMT-TR, F.Cu at (93.3, 73.7)
- added FID1: FIDUCIAL, Huey:FIDUCIAL, F.Cu at (58.4, 92.7)
- added FID2: FIDUCIAL, Huey:FIDUCIAL, F.Cu at (101.6, 73.7)
- added FID3: FIDUCIAL, Huey:FIDUCIAL, F.Cu at (94.6, 101.6)
- added MP1: MOUNTING_HOLE, Huey:MOUNTING_HOLE_#4, F.Cu at (59.0, 101.0)
- added MP2: MOUNTING_HOLE, Huey:MOUNTING_HOLE_#4, F.Cu at (101.0, 59.0)
- added MP3: MOUNTING_HOLE, Huey:MOUNTING_HOLE_#4, F.Cu at (59.0, 59.0)
- added MP4: MOUNTING_HOLE, Huey:MOUNTING_HOLE_#4, F.Cu at (101.0, 101.0)
- added P2: CONN_01X16, Huey:FEMALE_HEADER_16x1_SMD, F.Cu at (64.1, 77.5)
- added P3: CONN_01X12, Huey:FEMALE_HEADER_12x1_SMD, F.Cu at (85.1, 87.6)
- U1: value ADAFRUIT_FEATHER_M0_WIFI -> Adafruit_Feather_M0_WiFi
- moved R3 34.0 mm to (70.8, 74.5), turned to 0 degrees
- moved R4 32.5 mm to (79.1, 74.5), turned to 180 degrees
- moved R1 30.6 mm to (70.8, 77.1), turned to 180 degrees
- moved Q1 30.2 mm to (75.2, 76.5), turned to 90 degrees
- moved R2 29.0 mm to (79.1, 77.1), turned to 0 degrees
- moved SD1 15.8 mm to (74.9, 97.2), turned to 180 degrees
- moved P1 13.5 mm to (78.7, 65.4), turned to 270 degrees
- moved U1 8.89 mm to (74.3, 80.0)
Connections:
- R2 pad 2: Net-(R2-Pad2) -> Net-(P3-Pad10)
- SD1 pad 2: Net-(SD1-Pad2) -> Net-(P3-Pad7)
- SD1 pad 3: Net-(SD1-Pad3) -> Net-(P2-Pad12)
- SD1 pad 5: Net-(SD1-Pad5) -> Net-(P2-Pad11)
- SD1 pad 7: Net-(SD1-Pad7) -> Net-(P2-Pad13)
- U1 pad 11: Net-(SD1-Pad5) -> Net-(U1-Pad11)
- U1 pad 12: Net-(SD1-Pad3) -> Net-(U1-Pad12)
- U1 pad 13: Net-(SD1-Pad7) -> Net-(U1-Pad13)
- U1 pad 19: Net-(R2-Pad2) -> Net-(U1-Pad19)
- U1 pad 2: +3V3 -> Net-(U1-Pad2)
- U1 pad 22: Net-(SD1-Pad2) -> Net-(U1-Pad22)
Routing:
- net Net-(U1-Pad13): track 0.00 -> 1.21 mm
- net Net-(Q1-Pad2): track 0.00 -> 0.51 mm
- net Net-(Q1-Pad1): track 0.00 -> 0.51 mm
- added copper zone on B.Cu, net GND
- added copper zone on F.Cu, net GND
Other:
- outline, holes or cut-outs redrawn
- board text added: "HUEY Rev 1.0"
- board text added: "Kilo LLC"

Commit message: I think rev 1.0 is looking good... submitted for approval.
Parts:
- added P4: CONN_01X06, Pin_Headers:Pin_Header_Straight_1x06, F.Cu at (59.7, 72.4)
- added P5: CONN_01X02, Pin_Headers:Pin_Header_Straight_1x02, F.Cu at (59.7, 93.3)
- added P6: CONN_01X02, Pin_Headers:Pin_Header_Straight_1x02, F.Cu at (88.9, 97.8)
- FID1, FID2, FID3: footprint Huey:FIDUCIAL -> Fiducials:Fiducial_1mm_Dia_2.54mm_Outer_CopperTop
- P1: value LED_HEADERS -> TO_LEDS
- P2: value CONN_01X16 -> NPTC161KFXC-RC
- P3: value CONN_01X12 -> NPTC121KFXC-RC
- U1: value Adafruit_Feather_M0_WiFi -> FEATHER_M0_WIFI
- moved FID3 51.8 mm to (59.0, 64.0)
- moved FID1 50.9 mm to (101.0, 64.8)
- moved C1 29.7 mm to (92.0, 59.0), turned to 270 degrees
- moved FID2 28.5 mm to (95.9, 101.6)
- moved R3 8.58 mm to (79.4, 74.9), turned to 180 degrees
- moved CON1 8.26 mm to (96.5, 81.3)
- moved R4 7.95 mm to (71.1, 74.9), turned to 0 degrees
- moved P3 0.64 mm to (84.5, 87.6)
- moved R1 0.50 mm to (71.1, 77.5)
- moved R2 0.50 mm to (79.4, 77.5)
Connections:
- P2 pad 4: Net-(P2-Pad4) -> GND
- P3 pad 1: Net-(P3-Pad1) -> +5V
Routing:
- net +3V3: track 0.44 -> 44.9 mm
- net +5V: track 0.29 -> 42.9 mm
- net Net-(P3-Pad7): track 0.00 -> 21.4 mm
- net Net-(P2-Pad12): track 0.00 -> 21.0 mm, vias 0 -> 2
- net Net-(P3-Pad10): track 0.00 -> 19.8 mm, vias 0 -> 2
- net Net-(P2-Pad11): track 0.00 -> 17.8 mm
- net Net-(P1-Pad2): track 0.28 -> 13.3 mm
- net Net-(P2-Pad13): track 0.00 -> 12.7 mm
- net Net-(Q1-Pad3): track 0.00 -> 7.19 mm
- net Net-(P2-Pad15): track 0.00 -> 6.88 mm
- net Net-(P3-Pad12): track 0.00 -> 6.09 mm
- net Net-(P2-Pad9): track 0.00 -> 6.09 mm
- net Net-(P2-Pad7): track 0.00 -> 6.09 mm
- net Net-(P2-Pad5): track 0.00 -> 6.09 mm
- net Net-(SD1-Pad10): track 0.00 -> 5.83 mm, vias 0 -> 2
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