File: huey.sch (KiCad schematic (older format))
At the start: 4 parts

Commit message: starting layout
Parts:
- added Q1: MF-DSC-SOT233-BSS138, Huey:MF_Discrete_Semiconductor-SOT-23-3, symbol BSS138
- added R1, R2, R3, R4: MF-RES-0603-1K, Resistors_SMD:R_0603, symbol R
- P1: renamed from P?; footprint (none) -> Pin_Headers:Pin_Header_Straight_1x03
- SD1: renamed from SD?; footprint MF_Connectors_MF-MICROSD -> Huey:MF_Connectors-MF-MICROSD
- U1: renamed from U?; footprint (none) -> Huey:Adafruit_Feather_M0_WiFi
- gave numbers to parts that had none: 1
Connections:
- net +3V3: now also R1.2
- net +5V: now also R3.1
- net at U1.19 (D5): now also R2.2
- net at P1.2 (P2): now also R4.1
- new net: Q1.1 (G), R1.1
- new net: Q1.2 (S), R2.1
- new net: Q1.3 (D), R3.2, R4.2
Other:
- moved on the sheet: P1
Changed lines of the file:
@@
 LIBS:huey
 LIBS:MF_Connectors
+LIBS:huey-cache
 EELAYER 25 0
 EELAYER END
@@
 encoding utf-8
 Sheet 1 1
-Title ""
-Date ""
-Rev ""
-Comp ""
+Title "Huey Main Board"
+Date "2018-04-08"
+Rev "1.0"
+Comp "Kilo LLC"
 Comment1 ""
 Comment2 ""
@@
 $EndDescr
 $Comp
-L Adafruit_Feather_M0_WiFi U?
+L Adafruit_Feather_M0_WiFi U1
 U 1 1 5ACA666A
 P 6000 3950
-F 0 "U?" H 6000 4500 60  0000 C CNN
+F 0 "U1" H 6000 4500 60  0000 C CNN
 F 1 "Adafruit_Feather_M0_WiFi" V 6000 3800 60  0000 C CNN
-F 2 "" H 5850 3950 60  0001 C CNN
+F 2 "Huey:Adafruit_Feather_M0_WiFi" H 5850 3950 60  0001 C CNN
 F 3 "" H 5850 3950 60  0001 C CNN
 	1    6000 3950
@@
 $EndComp
 $Comp
-L SD_CARD_SLOT_MICRO_RIGHT SD?
+L SD_CARD_SLOT_MICRO_RIGHT SD1
 U 1 1 5ACAA1F7
 P 3200 3250
-F 0 "SD?" H 3200 3275 45  0000 L BNN
+F 0 "SD1" H 3200 3275 45  0000 L BNN
 F 1 "MF-MICROSD" V 3890 2050 45  0000 L BNN
-F 2 "MF_Connectors_MF-MICROSD" V 3940 2050 20  0001 L CNN
+F 2 "Huey:MF_Connectors-MF-MICROSD" V 3940 2050 20  0001 L CNN
 F 3 "" H 3200 3250 60  0000 C CNN
 	1    3200 3250
@@
 $EndComp
 $Comp
-L CONN_01X03 P?
+L CONN_01X03 P1
 U 1 1 5ACAA4AD
-P 9250 5650
-F 0 "P?" H 9250 5850 50  0000 C CNN
-F 1 "LED_HEADERS" V 9350 5650 50  0000 C CNN
-F 2 "" H 9250 5650 50  0000 C CNN
-F 3 "" H 9250 5650 50  0000 C CNN
-	1    9250 5650
-	1    0    0    -1
-$EndComp
-$Comp
-L BARREL_JACK CON?
+P 9850 4550
+F 0 "P1" H 9850 4750 50  0000 C CNN
+F 1 "LED_HEADERS" V 9950 4550 50  0000 C CNN
+F 2 "Pin_Headers:Pin_Header_Straight_1x03" H 9850 4550 50  0001 C CNN
+F 3 "" H 9850 4550 50  0000 C CNN
+	1    9850 4550
+	1    0    0    -1
+$EndComp
+$Comp
+L BARREL_JACK CON1
 U 1 1 5ACAA5F0
 P 3600 1700
-F 0 "CON?" H 3600 1950 50  0000 C CNN
+F 0 "CON1" H 3600 1950 50  0000 C CNN
 F 1 "BARREL_JACK" H 3600 1500 50  0000 C CNN
-F 2 "" H 3600 1700 50  0000 C CNN
+F 2 "" H 3600 1700 50  0001 C CNN
 F 3 "" H 3600 1700 50  0000 C CNN
 F 4 "CP-036AHPJCT-ND" H 3600 1700 60  0001 C CNN "Digikey Part"
@@
 $EndComp
 $Comp
-L +3.3V #PWR?
+L +3.3V #PWR01
 U 1 1 5ACAADCB
 P 2900 3050
-F 0 "#PWR?" H 2900 2900 50  0001 C CNN
+F 0 "#PWR01" H 2900 2900 50  0001 C CNN
 F 1 "+3.3V" H 2900 3190 50  0000 C CNN
 F 2 "" H 2900 3050 50  0000 C CNN
@@
 	2900 3050 2900 3150
 $Comp
-L +3.3V #PWR?
+L +3.3V #PWR02
 U 1 1 5ACAAF4B
 P 5150 3300
-F 0 "#PWR?" H 5150 3150 50  0001 C CNN
+F 0 "#PWR02" H 5150 3150 50  0001 C CNN
 F 1 "+3.3V" H 5150 3440 50  0000 C CNN
 F 2 "" H 5150 3300 50  0000 C CNN
@@
 	4700 3550 3300 3550
 $Comp
-L GND #PWR?
+L GND #PWR03
 U 1 1 5ACAB088
 P 2900 4650
-F 0 "#PWR?" H 2900 4400 50  0001 C CNN
+F 0 "#PWR03" H 2900 4400 50  0001 C CNN
 F 1 "GND" H 2900 4500 50  0000 C CNN
 F 2 "" H 2900 4650 50  0000 C CNN
@@
 	2900 4650 2900 4550
 $Comp
-L +5V #PWR?
+L +5V #PWR04
 U 1 1 5ACAB3F2
 P 4000 1600
-F 0 "#PWR?" H 4000 1450 50  0001 C CNN
+F 0 "#PWR04" H 4000 1450 50  0001 C CNN
 F 1 "+5V" H 4000 1740 50  0000 C CNN
 F 2 "" H 4000 1600 50  0000 C CNN
@@
 	4000 1600 3900 1600
 $Comp
-L GND #PWR?
+L GND #PWR05
 U 1 1 5ACAB49B
 P 4000 1800
-F 0 "#PWR?" H 4000 1550 50  0001 C CNN
+F 0 "#PWR05" H 4000 1550 50  0001 C CNN
 F 1 "GND" H 4000 1650 50  0000 C CNN
 F 2 "" H 4000 1800 50  0000 C CNN
@@
 NoConn ~ 3900 1700
 $Comp
-L +5V #PWR?
+L +5V #PWR06
 U 1 1 5ACAB6CE
-P 8950 5550
-F 0 "#PWR?" H 8950 5400 50  0001 C CNN
-F 1 "+5V" H 8950 5690 50  0000 C CNN
-F 2 "" H 8950 5550 50  0000 C CNN
-F 3 "" H 8950 5550 50  0000 C CNN
-	1    8950 5550
-	0    -1   -1   0
-$EndComp
-Wire Wire Line
-	9050 5550 8950 5550
-$Comp
-L GND #PWR?
+P 9550 4450
+F 0 "#PWR06" H 9550 4300 50  0001 C CNN
+F 1 "+5V" H 9550 4590 50  0000 C CNN
+F 2 "" H 9550 4450 50  0000 C CNN
+F 3 "" H 9550 4450 50  0000 C CNN
+	1    9550 4450
+	0    -1   -1   0
+$EndComp
+Wire Wire Line
+	9650 4450 9550 4450
+$Comp
+L GND #PWR07
 U 1 1 5ACAB70E
-P 8950 5750
-F 0 "#PWR?" H 8950 5500 50  0001 C CNN
-F 1 "GND" H 8950 5600 50  0000 C CNN
-F 2 "" H 8950 5750 50  0000 C CNN
-F 3 "" H 8950 5750 50  0000 C CNN
-	1    8950 5750
-	0    1    1    0
-$EndComp
-Wire Wire Line
-	9050 5750 8950 5750
+P 9550 4650
+F 0 "#PWR07" H 9550 4400 50  0001 C CNN
+F 1 "GND" H 9550 4500 50  0000 C CNN
+F 2 "" H 9550 4650 50  0000 C CNN
+F 3 "" H 9550 4650 50  0000 C CNN
+	1    9550 4650
+	0    1    1    0
+$EndComp
+Wire Wire Line
+	9650 4650 9550 4650
+$Comp
+L BSS138 Q1
+U 1 1 5ACA7902
+P 8300 4800
+F 0 "Q1" H 8500 4875 50  0000 L CNN
+F 1 "MF-DSC-SOT233-BSS138" H 8500 4800 50  0000 L CNN
+F 2 "Huey:MF_Discrete_Semiconductor-SOT-23-3" H 8500 4725 50  0001 L CIN
+F 3 "" H 8300 4800 50  0000 L CNN
+	1    8300 4800
+	1    0    0    -1
+$EndComp
+Wire Wire Line
+	8400 4500 8400 4600
+$Comp
+L R R3
+U 1 1 5ACA7BF6
+P 8400 4350
+F 0 "R3" V 8480 4350 50  0000 C CNN
+F 1 "MF-RES-0603-1K" V 8400 4350 50  0000 C CNN
+F 2 "Resistors_SMD:R_0603" V 8330 4350 50  0001 C CNN
+F 3 "" H 8400 4350 50  0000 C CNN
+	1    8400 4350
+	1    0    0    -1
+$EndComp
+$Comp
+L +5V #PWR08
+U 1 1 5ACA7E2D
+P 8400 4100
+F 0 "#PWR08" H 8400 3950 50  0001 C CNN
+F 1 "+5V" H 8400 4240 50  0000 C CNN
+F 2 "" H 8400 4100 50  0000 C CNN
+F 3 "" H 8400 4100 50  0000 C CNN
+	1    8400 4100
+	1    0    0    -1
+$EndComp
+Wire Wire Line
+	8400 4100 8400 4200
+Connection ~ 8400 4550
+Wire Wire Line
+	6750 4500 7200 4500
+Wire Wire Line
+	7200 4500 7200 5250
+Wire Wire Line
+	8400 5250 8400 5000
+$Comp
+L R R1
+U 1 1 5ACA80D2
+P 7850 4850
+F 0 "R1" V 7930 4850 50  0000 C CNN
+F 1 "MF-RES-0603-1K" V 7850 4850 50  0000 C CNN
+F 2 "Resistors_SMD:R_0603" V 7780 4850 50  0001 C CNN
+F 3 "" H 7850 4850 50  0000 C CNN
+	1    7850 4850
+	0    1    1    0
+$EndComp
+Wire Wire Line
+	8000 4850 8100 4850
+$Comp
+L +3.3V #PWR09
+U 1 1 5ACA814D
+P 7600 4850
+F 0 "#PWR09" H 7600 4700 50  0001 C CNN
+F 1 "+3.3V" H 7600 4990 50  0000 C CNN
+F 2 "" H 7600 4850 50  0000 C CNN
+F 3 "" H 7600 4850 50  0000 C CNN
+	1    7600 4850
+	0    -1   -1   0
+$EndComp
+Wire Wire Line
+	7600 4850 7700 4850
+$Comp
+L R R2
+U 1 1 5ACA81AB
+P 8150 5250
+F 0 "R2" V 8230 5250 50  0000 C CNN
+F 1 "MF-RES-0603-1K" V 8150 5250 50  0000 C CNN
+F 2 "Resistors_SMD:R_0603" V 8080 5250 50  0001 C CNN
+F 3 "" H 8150 5250 50  0000 C CNN
+	1    8150 5250
+	0    1    1    0
+$EndComp
+Wire Wire Line
+	8300 5250 8400 5250
+Wire Wire Line
+	7200 5250 8000 5250
+$Comp
+L R R4
+U 1 1 5ACA84D7
+P 8950 4550
+F 0 "R4" V 9030 4550 50  0000 C CNN
+F 1 "MF-RES-0603-1K" V 8950 4550 50  0000 C CNN
+F 2 "Resistors_SMD:R_0603" V 8880 4550 50  0001 C CNN
+F 3 "" H 8950 4550 50  0000 C CNN
+	1    8950 4550
+	0    1    1    0
+$EndComp
+Wire Wire Line
+	8400 4550 8800 4550
+Wire Wire Line
+	9100 4550 9650 4550
 $EndSCHEMATC

Commit message: WIP
Parts:
- added C1: MF-CAP-6.3MM-100uF, Huey:MF_Passives-CP6.3MM, symbol CP
- added FID1, FID2, FID3: FIDUCIAL, Huey:FIDUCIAL, symbol MOUNTING_HOLE
- added MP1, MP2, MP3, MP4: MOUNTING_HOLE, Huey:MOUNTING_HOLE_#4, symbol MOUNTING_HOLE
- added P2: CONN_01X16, Huey:FEMALE_HEADER_16x1_SMD, symbol CONN_01X16
- added P3: CONN_01X12, Huey:FEMALE_HEADER_12x1_SMD, symbol CONN_01X12
- CON1: footprint (none) -> Huey:PJ-036AH-SMT-TR
Connections:
- net +3V3: now also P2.2 (P2); no longer U1.2 (3V3)
- net +5V: now also C1.1
- net GND: now also C1.2, MP1.1 (GND), MP2.1 (GND), MP3.1 (GND), MP4.1 (GND)
- net at U1.11 (D24/SCK): no longer SD1.5 (SCLK)
- net at U1.12 (D23/MOSI): no longer SD1.3 (DI)
- net at U1.13 (D22/MISO): no longer SD1.7 (D0)
- net at U1.19 (D5): no longer R2.2
- net at U1.22 (D10): no longer SD1.2 (CS)
- new net: P3.10 (P10), R2.2
- new net: P3.7 (P7), SD1.2 (CS)
- new net: P2.12 (P12), SD1.3 (DI)
- new net: P2.11 (P11), SD1.5 (SCLK)
- new net: P2.13 (P13), SD1.7 (D0)
- no-connect marks 3 -> 4
Changed lines of the file:
@@
 F 0 "CON1" H 3600 1950 50  0000 C CNN
 F 1 "BARREL_JACK" H 3600 1500 50  0000 C CNN
-F 2 "" H 3600 1700 50  0001 C CNN
+F 2 "Huey:PJ-036AH-SMT-TR" H 3600 1700 50  0001 C CNN
 F 3 "" H 3600 1700 50  0000 C CNN
 F 4 "CP-036AHPJCT-ND" H 3600 1700 60  0001 C CNN "Digikey Part"
@@
 L +3.3V #PWR02
 U 1 1 5ACAAF4B
-P 5150 3300
-F 0 "#PWR02" H 5150 3150 50  0001 C CNN
-F 1 "+3.3V" H 5150 3440 50  0000 C CNN
-F 2 "" H 5150 3300 50  0000 C CNN
-F 3 "" H 5150 3300 50  0000 C CNN
-	1    5150 3300
+P 4850 3300
+F 0 "#PWR02" H 4850 3150 50  0001 C CNN
+F 1 "+3.3V" H 4850 3440 50  0000 C CNN
+F 2 "" H 4850 3300 50  0000 C CNN
+F 3 "" H 4850 3300 50  0000 C CNN
+	1    4850 3300
 	0    -1   -1   0
 $EndComp
 Wire Wire Line
-	5150 3300 5250 3300
-NoConn ~ 5250 3200
-NoConn ~ 5250 3400
-Wire Wire Line
-	5250 4400 4600 4400
-Wire Wire Line
 	4600 4400 4600 3850
 Wire Wire Line
@@
 	4700 3650 4700 4300
 Wire Wire Line
-	4700 4300 5250 4300
-Wire Wire Line
-	5250 4200 4800 4200
-Wire Wire Line
 	4800 4200 4800 3750
 Wire Wire Line
 	4800 3750 3300 3750
-Wire Wire Line
-	6750 4200 8150 4200
 Wire Wire Line
 	8150 4200 8150 2650
@@
 L +5V #PWR04
 U 1 1 5ACAB3F2
-P 4000 1600
-F 0 "#PWR04" H 4000 1450 50  0001 C CNN
-F 1 "+5V" H 4000 1740 50  0000 C CNN
-F 2 "" H 4000 1600 50  0000 C CNN
-F 3 "" H 4000 1600 50  0000 C CNN
-	1    4000 1600
-	0    1    1    0
-$EndComp
-Wire Wire Line
-	4000 1600 3900 1600
+P 4500 1600
+F 0 "#PWR04" H 4500 1450 50  0001 C CNN
+F 1 "+5V" H 4500 1740 50  0000 C CNN
+F 2 "" H 4500 1600 50  0000 C CNN
+F 3 "" H 4500 1600 50  0000 C CNN
+	1    4500 1600
+	0    1    1    0
+$EndComp
+Wire Wire Line
+	3900 1600 4500 1600
 $Comp
 L GND #PWR05
 U 1 1 5ACAB49B
-P 4000 1800
-F 0 "#PWR05" H 4000 1550 50  0001 C CNN
-F 1 "GND" H 4000 1650 50  0000 C CNN
-F 2 "" H 4000 1800 50  0000 C CNN
-F 3 "" H 4000 1800 50  0000 C CNN
-	1    4000 1800
+P 4500 2000
+F 0 "#PWR05" H 4500 1750 50  0001 C CNN
+F 1 "GND" H 4500 1850 50  0000 C CNN
+F 2 "" H 4500 2000 50  0000 C CNN
+F 3 "" H 4500 2000 50  0000 C CNN
+	1    4500 2000
 	0    -1   -1   0
 $EndComp
-Wire Wire Line
-	4000 1800 3900 1800
 NoConn ~ 3900 1700
 $Comp
@@
 P 8400 4350
 F 0 "R3" V 8480 4350 50  0000 C CNN
-F 1 "MF-RES-0603-1K" V 8400 4350 50  0000 C CNN
+F 1 "MF-RES-0603-1K" V 8300 4450 50  0000 C CNN
 F 2 "Resistors_SMD:R_0603" V 8330 4350 50  0001 C CNN
 F 3 "" H 8400 4350 50  0000 C CNN
@@
 Connection ~ 8400 4550
 Wire Wire Line
-	6750 4500 7200 4500
-Wire Wire Line
 	7200 4500 7200 5250
 Wire Wire Line
@@
 P 7850 4850
 F 0 "R1" V 7930 4850 50  0000 C CNN
-F 1 "MF-RES-0603-1K" V 7850 4850 50  0000 C CNN
+F 1 "MF-RES-0603-1K" V 7750 4850 50  0000 C CNN
 F 2 "Resistors_SMD:R_0603" V 7780 4850 50  0001 C CNN
 F 3 "" H 7850 4850 50  0000 C CNN
@@
 P 8150 5250
 F 0 "R2" V 8230 5250 50  0000 C CNN
-F 1 "MF-RES-0603-1K" V 8150 5250 50  0000 C CNN
+F 1 "MF-RES-0603-1K" V 8050 5100 50  0000 C CNN
 F 2 "Resistors_SMD:R_0603" V 8080 5250 50  0001 C CNN
 F 3 "" H 8150 5250 50  0000 C CNN
@@
 P 8950 4550
 F 0 "R4" V 9030 4550 50  0000 C CNN
-F 1 "MF-RES-0603-1K" V 8950 4550 50  0000 C CNN
+F 1 "MF-RES-0603-1K" V 8850 4550 50  0000 C CNN
 F 2 "Resistors_SMD:R_0603" V 8880 4550 50  0001 C CNN
 F 3 "" H 8950 4550 50  0000 C CNN
@@
 Wire Wire Line
 	9100 4550 9650 4550
+$Comp
+L MOUNTING_HOLE MP1
+U 1 1 5ACA83D6
+P 5250 5750
+F 0 "MP1" H 5250 5650 20  0000 C CNN
+F 1 "MOUNTING_HOLE" H 5250 5850 20  0000 C CNN
+F 2 "Huey:MOUNTING_HOLE_#4" H 5250 5750 60  0001 C CNN
+F 3 "" H 5250 5750 60  0000 C CNN
+	1    5250 5750
+	1    0    0    -1
+$EndComp
+$Comp
+L MOUNTING_HOLE MP3
+U 1 1 5ACA866B
+P 5250 6350
+F 0 "MP3" H 5250 6250 20  0000 C CNN
+F 1 "MOUNTING_HOLE" H 5250 6450 20  0000 C CNN
+F 2 "Huey:MOUNTING_HOLE_#4" H 5250 6350 60  0001 C CNN
+F 3 "" H 5250 6350 60  0000 C CNN
+	1    5250 6350
+	1    0    0    -1
+$EndComp
+$Comp
+L MOUNTING_HOLE MP4
+U 1 1 5ACA86A8
+P 5250 6650
+F 0 "MP4" H 5250 6550 20  0000 C CNN
+F 1 "MOUNTING_HOLE" H 5250 6750 20  0000 C CNN
+F 2 "Huey:MOUNTING_HOLE_#4" H 5250 6650 60  0001 C CNN
+F 3 "" H 5250 6650 60  0000 C CNN
+	1    5250 6650
+	1    0    0    -1
+$EndComp
+$Comp
+L MOUNTING_HOLE MP2
+U 1 1 5ACA8704
+P 5250 6050
+F 0 "MP2" H 5250 5950 20  0000 C CNN
+F 1 "MOUNTING_HOLE" H 5250 6150 20  0000 C CNN
+F 2 "Huey:MOUNTING_HOLE_#4" H 5250 6050 60  0001 C CNN
+F 3 "" H 5250 6050 60  0000 C CNN
+	1    5250 6050
+	1    0    0    -1
+$EndComp
+$Comp
+L CP C1
+U 1 1 5ACACF6F
+P 4250 1800
+F 0 "C1" H 4275 1900 50  0000 L CNN
+F 1 "MF-CAP-6.3MM-100uF" H 4400 1800 50  0000 L CNN
+F 2 "Huey:MF_Passives-CP6.3MM" H 4288 1650 50  0001 C CNN
+F 3 "" H 4250 1800 50  0000 C CNN
+	1    4250 1800
+	1    0    0    -1
+$EndComp
+Wire Wire Line
+	4250 1650 4250 1600
+Connection ~ 4250 1600
+Wire Wire Line
+	3900 1800 4050 1800
+Wire Wire Line
+	4050 1800 4050 2000
+Wire Wire Line
+	4050 2000 4500 2000
+Wire Wire Line
+	4250 2000 4250 1950
+Connection ~ 4250 2000
+$Comp
+L MOUNTING_HOLE FID1
+U 1 1 5ACB2643
+P 6050 6100
+F 0 "FID1" H 6050 6000 20  0000 C CNN
+F 1 "FIDUCIAL" H 6050 6200 20  0000 C CNN
+F 2 "Huey:FIDUCIAL" H 6050 6100 60  0001 C CNN
+F 3 "" H 6050 6100 60  0000 C CNN
+	1    6050 6100
+	1    0    0    -1
+$EndComp
+$Comp
+L MOUNTING_HOLE FID2
+U 1 1 5ACB26A6
+P 6300 6100
+F 0 "FID2" H 6300 6000 20  0000 C CNN
+F 1 "FIDUCIAL" H 6300 6200 20  0000 C CNN
+F 2 "Huey:FIDUCIAL" H 6300 6100 60  0001 C CNN
+F 3 "" H 6300 6100 60  0000 C CNN
+	1    6300 6100
+	1    0    0    -1
+$EndComp
+$Comp
+L MOUNTING_HOLE FID3
+U 1 1 5ACB26F2
+P 6550 6100
+F 0 "FID3" H 6550 6000 20  0000 C CNN
+F 1 "FIDUCIAL" H 6550 6200 20  0000 C CNN
+F 2 "Huey:FIDUCIAL" H 6550 6100 60  0001 C CNN
+F 3 "" H 6550 6100 60  0000 C CNN
+	1    6550 6100
+	1    0    0    -1
+$EndComp
+NoConn ~ 5950 6100
+NoConn ~ 6200 6100
+NoConn ~ 6450 6100
+$Comp
+L GND #PWR010
+U 1 1 5ACB297A
+P 5050 6750
+F 0 "#PWR010" H 5050 6500 50  0001 C CNN
+F 1 "GND" H 5050 6600 50  0000 C CNN
+F 2 "" H 5050 6750 50  0000 C CNN
+F 3 "" H 5050 6750 50  0000 C CNN
+	1    5050 6750
+	1    0    0    -1
+$EndComp
+Wire Wire Line
+	5050 5750 5050 6750
+Wire Wire Line
+	5050 6050 5150 6050
+Wire Wire Line
+	5050 5750 5150 5750
+Connection ~ 5050 6050
+Wire Wire Line
+	5050 6650 5150 6650
+Connection ~ 5050 6650
+Wire Wire Line
+	5150 6350 5050 6350
+Connection ~ 5050 6350
+$Comp
+L CONN_01X16 P2
+U 1 1 5ACB3909
+P 5150 3950
+F 0 "P2" H 5150 4800 50  0000 C CNN
+F 1 "CONN_01X16" H 5000 3100 50  0000 C CNN
+F 2 "Huey:FEMALE_HEADER_16x1_SMD" H 5150 3950 50  0001 C CNN
+F 3 "" H 5150 3950 50  0000 C CNN
+	1    5150 3950
+	1    0    0    -1
+$EndComp
+Wire Wire Line
+	4850 3300 4950 3300
+Wire Wire Line
+	4800 4200 4950 4200
+Wire Wire Line
+	4700 4300 4950 4300
+Wire Wire Line
+	4600 4400 4950 4400
+$Comp
+L CONN_01X12 P3
+U 1 1 5ACB3E04
+P 6900 4150
+F 0 "P3" H 6900 4800 50  0000 C CNN
+F 1 "CONN_01X12" H 6900 3500 50  0000 C CNN
+F 2 "Huey:FEMALE_HEADER_12x1_SMD" H 6900 4150 50  0001 C CNN
+F 3 "" H 6900 4150 50  0000 C CNN
+	1    6900 4150
+	-1   0    0    -1
+$EndComp
+Wire Wire Line
+	7100 4500 7200 4500
+Wire Wire Line
+	8150 4200 7100 4200
 $EndSCHEMATC
