File: _saved_huey.sch (KiCad schematic (older format))
At the start: 22 parts, among them CON1 BARREL_JACK, P1 TO_LEDS, P2 NPTC161KFXC-RC, P3 NPTC121KFXC-RC, Q1 MF-DSC-SOT233-BSS138, U1 FEATHER_M0_WIFI

Commit message: I think rev 1.0 is looking good... submitted for approval.
Parts:
- P4: renamed from P?; footprint (none) -> Pin_Headers:Pin_Header_Straight_1x06
- P5, P6: renamed from P?; footprint (none) -> Pin_Headers:Pin_Header_Straight_1x02
Changed lines of the file:
@@
 	7100 3600 7200 3600
 $Comp
-L +5V #PWR?
+L +5V #PWR011
 U 1 1 5ACB5DED
 P 7200 3600
-F 0 "#PWR?" H 7200 3450 50  0001 C CNN
+F 0 "#PWR011" H 7200 3450 50  0001 C CNN
 F 1 "+5V" H 7200 3740 50  0000 C CNN
 F 2 "" H 7200 3600 50  0000 C CNN
@@
 $EndComp
 $Comp
-L CONN_01X02 P?
+L CONN_01X02 P5
 U 1 1 5ACB61B2
 P 4300 4550
-F 0 "P?" H 4300 4700 50  0000 C CNN
+F 0 "P5" H 4300 4700 50  0000 C CNN
 F 1 "CONN_01X02" V 4400 4550 50  0000 C CNN
-F 2 "" H 4300 4550 50  0000 C CNN
+F 2 "Pin_Headers:Pin_Header_Straight_1x02" H 4300 4550 50  0001 C CNN
 F 3 "" H 4300 4550 50  0000 C CNN
 	1    4300 4550
@@
 	4500 4600 4950 4600
 $Comp
-L CONN_01X02 P?
+L CONN_01X02 P6
 U 1 1 5ACB6614
 P 7850 4450
-F 0 "P?" H 7850 4600 50  0000 C CNN
+F 0 "P6" H 7850 4600 50  0000 C CNN
 F 1 "CONN_01X02" V 7950 4450 50  0000 C CNN
-F 2 "" H 7850 4450 50  0000 C CNN
+F 2 "Pin_Headers:Pin_Header_Straight_1x02" H 7850 4450 50  0001 C CNN
 F 3 "" H 7850 4450 50  0000 C CNN
 	1    7850 4450
@@
 	4950 3500 4850 3500
 $Comp
-L GND #PWR?
+L GND #PWR012
 U 1 1 5ACB686A
 P 4850 3500
-F 0 "#PWR?" H 4850 3250 50  0001 C CNN
+F 0 "#PWR012" H 4850 3250 50  0001 C CNN
 F 1 "GND" H 4850 3350 50  0000 C CNN
 F 2 "" H 4850 3500 50  0000 C CNN
@@
 $EndComp
 $Comp
-L CONN_01X06 P?
+L CONN_01X06 P4
 U 1 1 5ACB68A1
 P 4300 3850
-F 0 "P?" H 4300 4200 50  0000 C CNN
+F 0 "P4" H 4300 4200 50  0000 C CNN
 F 1 "CONN_01X06" V 4400 3850 50  0000 C CNN
-F 2 "" H 4300 3850 50  0000 C CNN
+F 2 "Pin_Headers:Pin_Header_Straight_1x06" H 4300 3850 50  0001 C CNN
 F 3 "" H 4300 3850 50  0000 C CNN
 	1    4300 3850
